Commit message: modified xacro

File: missions/params/giraff.xacro (robot description, xacro)
@@ -25,5 +25,5 @@
     <color rgba="0.0 0.9 0.0 1"/>
   </material>
-  # Base
+  # Base_link
   <link name="$(arg frame_ns)_base_link">
     <visual>
@@ -32,5 +32,5 @@
       </geometry>
       <material name="blue"/>
-      <origin xyz="0 0 0.15"/>
+      <origin xyz="0 0 0.1"/>
     </visual>
   </link>

Commit message: added new tf xacro

File: missions/params/giraff.xacro (robot description, xacro)
@@ -1,10 +1,16 @@
-<?xml version="1.0" ?>
-<!-- =================================================================================== -->
-<!-- |    This document was autogenerated by xacro from giraff.urdf                    | -->
-<!-- |    EDITING THIS FILE BY HAND IS NOT RECOMMENDED                                 | -->
-<!-- =================================================================================== -->
+<!--
+ URDF MODEL of GIRAFF-X
+ - Here we set Fixed and movable joints
+ - To move the parts in RVIZ, publish sensor_msgs/JointState messages.
+ - robot_state_publisher node calculates all of transforms between the different parts.
+ - The resulting transform tree is then used to display all of the shapes in Rviz.
+-->
+<?xml version="1.0"?>
 <robot xmlns:xacro="http://www.ros.org/wiki/xacro" name="giraff">
-  <xacro:arg name="frame_ns" default="giraff"/>
+<xacro:arg name="frame_ns" default="giraff"/>
   ### Define colors
+  <material name="body_color">
+    <color rgba="0.01 0.37 0.14 1"/>
+  </material>
   <material name="blue">
     <color rgba="0.41 0.83 0.96 1"/>
@@ -16,5 +22,5 @@
     <color rgba="1 1 1 1"/>
   </material>
-  <material name="grey">
+    <material name="grey">
     <color rgba="0.5 0.5 0.5 1"/>
   </material>
@@ -25,103 +31,121 @@
     <color rgba="0.0 0.9 0.0 1"/>
   </material>
-  # Base_link
-  <link name="$(arg frame_ns)_base_link">
-    <visual>
-      <geometry>
-        <cylinder length="0.23" radius="0.26"/>
-      </geometry>
-      <material name="blue"/>
-      <origin xyz="0 0 0.1"/>
-    </visual>
-  </link>
+  # Base
+  <link name="base_link">
+    <visual>
+      <geometry>
+        <cylinder length="0.20" radius="0.26"/>
+      </geometry>
+      <material name="body_color"/>
+      <origin rpy="0 0 0" xyz="0 0 0.13"/>              # Displacement/rotation of the part center with respect the reference_link (base_link)
+    </visual>
+  </link>
+  # Left wheel
+  <link name="left_wheel">
+    <visual>
+      <origin rpy="1.57075 0 0" xyz="0 0 0"/>           # Displacement/rotation of the part center with respect the reference_link
+      <geometry>
+        <cylinder length="0.02" radius="0.10"/>
+      </geometry>
+      <material name="black"/>
+    </visual>
+  </link>
+  <joint name="base_to_left_wheel_joint" type="fixed">
+    <parent link="base_link"/>
+    <child link="left_wheel"/>
+    <origin rpy="0 0 0" xyz="0 0.24 0.10"/>             # Displacement/rotation of the reference_link with respect parent reference_link (TF)
+  </joint>
   # Right wheel
-  <link name="$(arg frame_ns)_right_wheel">
-    <visual>
-      <origin rpy="1.57075 0 0" xyz="0 0 0"/>
-      <geometry>
-        <cylinder length="0.03" radius="0.10"/>
-      </geometry>
-      <material name="black"/>
-    </visual>
-  </link>
-  <joint name="$(arg frame_ns)_base_to_right_wheel_joint" type="fixed">
-    <parent link="$(arg frame_ns)_base_link"/>
-    <child link="$(arg frame_ns)_right_wheel"/>
-    <origin rpy="0 0 0" xyz="0 0.26 0.1"/>
-  </joint>
-  #Left wheel
-  <link name="$(arg frame_ns)_left_wheel">
-    <visual>
-      <origin rpy="1.57075 0 0" xyz="0 0 0"/>
-      <geometry>
-        <cylinder length="0.03" radius="0.10"/>
-      </geometry>
-      <material name="black"/>
-    </visual>
-  </link>
-  <joint name="$(arg frame_ns)_base_to_left_wheel_joint" type="fixed">
-    <parent link="$(arg frame_ns)_base_link"/>
-    <child link="$(arg frame_ns)_left_wheel"/>
-    <origin rpy="0 0 0" xyz="0 -0.26 0.1"/>
+  <link name="right_wheel">
+    <visual>
+      <origin rpy="1.57075 0 0" xyz="0 0 0"/>           # Displacement/rotation of the part center with respect the reference_link
+      <geometry>
+        <cylinder length="0.02" radius="0.10"/>
+      </geometry>
+      <material name="black"/>
+    </visual>
+  </link>
+  <joint name="base_to_right_wheel_joint" type="fixed">
+    <parent link="base_link"/>
+    <child link="right_wheel"/>
+    <origin rpy="0 0 0" xyz="0 -0.24 0.10"/>            # Displacement/rotation of the reference_link with respect parent reference_link (TF)
   </joint>
   # Body
-  <link name="$(arg frame_ns)_body">
-    <visual>
-      <geometry>
-        <box size="0.3 0.2 0.45"/>
-      </geometry>
-      <material name="blue"/>
-    </visual>
-  </link>
-  <joint name="$(arg frame_ns)_base_to_body" type="fixed">
-    <parent link="$(arg frame_ns)_base_link"/>
-    <child link="$(arg frame_ns)_body"/>
+  <link name="body">
+    <visual>
+      <geometry>
+        <box size="0.30 0.20 0.45"/>
+      </geometry>
+      <material name="body_color"/>
+    </visual>
+  </link>
+  <joint name="base_to_body" type="fixed">
+    <parent link="base_link"/>
+    <child link="body"/>
     <origin xyz="0.0 0.0 0.455"/>
   </joint>
-  #Neck
-  <link name="$(arg frame_ns)_neck">
-    <visual>
-      <geometry>
-        <box size="0.05 0.05 0.45"/>
+  # Neck (this tf is considered fixed)
+  <link name="neck">
+    <visual>
+      <geometry>
+        <box size="0.05 0.05 0.41"/>
       </geometry>
       <material name="grey"/>
     </visual>
   </link>
-  <joint name="$(arg frame_ns)_body_to_neck" type="fixed">
-    <parent link="$(arg frame_ns)_body"/>
-    <child link="$(arg frame_ns)_neck"/>
-    <origin xyz="0.0 0.0 0.45"/>
-  </joint>
-  #Head
-  <link name="$(arg frame_ns)_head">
-    <visual>
-      <geometry>
-        <box size="0.05 0.23 0.38"/>
-      </geometry>
-      <material name="blue"/>
-    </visual>
-  </link>
-  <joint name="$(arg frame_ns)_neck_to_head" type="fixed">
-    <parent link="$(arg frame_ns)_neck"/>
-    <child link="$(arg frame_ns)_head"/>
-    <origin xyz="0 0 0.415"/>
-  </joint>
-  #Screen
-  <link name="$(arg frame_ns)_screen">
-    <visual>
-      <geometry>
-        <box size="0.05 0.21 0.36"/>
+  <joint name="body_to_neck" type="fixed">
+    <parent link="body"/>
+    <child link="neck"/>
+    <origin xyz="0.0 0.0 0.43"/>
+  </joint>
+  # Head
+  <link name="head">
+    <visual>
+      <geometry>
+        <box size="0.05 0.30 0.56"/>
+      </geometry>
+      <material name="body_color"/>
+    </visual>
+  </link>
+  <joint name="neck_to_head" type="fixed">
+    <parent link="neck"/>
+    <child link="head"/>
+    <origin xyz="0 0 0.485"/>
+  </joint>
+  # Screen (this tf is published by the giraff_ros_driver using Tilt)
+  <link name="screen">
+    <visual>
+      <geometry>
+        <box size="0.05 0.22 0.40"/>
       </geometry>
       <material name="white"/>
     </visual>
   </link>
-  <joint name="$(arg frame_ns)_head_to_screen" type="fixed">
-    <parent link="$(arg frame_ns)_head"/>
-    <child link="$(arg frame_ns)_screen"/>
-    <origin xyz="0.02 0.0 0.0"/>
-  </joint>
-  ## EXTRAS ##
-  #Hokuyo front
-  <link name="$(arg frame_ns)_hokuyo_front">
+  <joint name="neck_to_screen" type="revolute">
+    <parent link="head"/>
+    <child link="screen"/>
+    <axis xyz="0 1 0"/>
+    <limit effort="1000.0" lower="-2.094395102" upper="2.094395102" velocity="0.5"/>
+    <origin rpy="0 0 0" xyz="0.02 0.0 0.0"/>
+  </joint>
+  ## SENSORS AND ACTUATORS ##
+  #=========================#
+  # FISH_EYE
+  <link name="usb_camera_link">
+    <visual>
+      <geometry>
+        <cylinder length="0.02" radius="0.02"/>
+      </geometry>
+      <material name="black"/>
+      <origin rpy="0 1.57079 0" xyz="0 0.0 0.0"/>     # Displacement/Rotation of the center with respect usb_camera_link
+    </visual>
+  </link>
+  <joint name="screen_to_usb_camera_link" type="fixed">
+    <parent link="screen"/>
+    <child link="usb_camera_link"/>
+    <origin rpy="0 0.3927 0" xyz="0.05 0.0 0.20"/>
+  </joint>
+  # Hokuyo front
+  <link name="laser_link">
     <visual>
       <geometry>
@@ -129,13 +153,47 @@
       </geometry>
       <material name="black"/>
-    </visual>
-  </link>
-  <joint name="$(arg frame_ns)_base_to_hokuyo_front" type="fixed">
-    <parent link="$(arg frame_ns)_base_link"/>
-    <child link="$(arg frame_ns)_hokuyo_front"/>
-    <origin xyz="0.2 0.0 0.28"/>
-  </joint>
-  #red button
-  <link name="$(arg frame_ns)_red_button">
+      <origin rpy="0 0 0" xyz="0 0.0 -0.03"/>     # Displacement/Rotation of the center with respect laser_link
+    </visual>
+  </link>
+  <joint name="base_link_to_laser_link" type="fixed">
+    <parent link="base_link"/>
+    <child link="laser_link"/>
+    <origin rpy="0 0 0" xyz="0.2062 0.0 0.0"/>     # Set Manually z=0.28
+  </joint>
+  # RGBD_DOWN
+  # For ASTRA rgbd cameras ref_link is located 10cm in y-axis
+  <link name="camera_down_link">
+    <visual>
+      <geometry>
+        <box size="0.04 0.16 0.03"/>
+      </geometry>
+      <material name="black"/>
+      <origin rpy="0 0 0" xyz="0 -0.10 0.0"/>     # Displacement/Rotation of the center with respect camera_down_link
+    </visual>
+  </link>
+  <joint name="base_link_to_camera_down_link" type="fixed">
+    <parent link="base_link"/>
+    <child link="camera_down_link"/>
+    <origin rpy="0 -0.2 0" xyz="0.06 0.10 0.985"/>     # Manually set
+  </joint>
+  # RGBD_UP
+  # For ASTRA rgbd cameras ref_link is located 10cm in y-axis
+  <link name="camera_up_link">
+    <visual>
+      <geometry>
+        <box size="0.04 0.16 0.03"/>
+      </geometry>
+      <material name="black"/>
+      <origin rpy="0 0 0" xyz="0 -0.06 0.0"/>     # Displacement/Rotation of the center with respect camera_up_link
+    </visual>
+  </link>
+  <joint name="base_link_to_camera_up_link" type="fixed">
+    <parent link="base_link"/>
+    <child link="camera_up_link"/>
+    <!-- <origin rpy="0 0.8 0" xyz="0.09 0.10 1.65"/> -->     # Manually set
+    <origin rpy="0.0062 0.7527 0" xyz="0.09 0.06 1.5737"/>             # Calibration
+  </joint>
+  # red button
+  <link name="red_button">
     <visual>
       <geometry>
@@ -145,11 +203,11 @@
     </visual>
   </link>
-  <joint name="$(arg frame_ns)_body_to_red_button" type="fixed">
-    <parent link="$(arg frame_ns)_body"/>
-    <child link="$(arg frame_ns)_red_button"/>
+  <joint name="body_to_red_button" type="fixed">
+    <parent link="body"/>
+    <child link="red_button"/>
     <origin xyz="0.11 0.05 0.225"/>
   </joint>
-  #green button
-  <link name="$(arg frame_ns)_green_button">
+  # green button
+  <link name="green_button">
     <visual>
       <geometry>
@@ -159,8 +217,22 @@
     </visual>
   </link>
-  <joint name="$(arg frame_ns)_body_to_green_button" type="fixed">
-    <parent link="$(arg frame_ns)_body"/>
-    <child link="$(arg frame_ns)_green_button"/>
+  <joint name="body_to_green_button" type="fixed">
+    <parent link="body"/>
+    <child link="green_button"/>
     <origin xyz="0.11 -0.05 0.225"/>
   </joint>
+  # e-stop button
+  <link name="estop_button">
+    <visual>
+      <geometry>
+        <cylinder length="0.02" radius="0.02"/>
+      </geometry>
+      <material name="red"/>
+    </visual>
+  </link>
+  <joint name="body_to_estop_button" type="fixed">
+    <parent link="body"/>
+    <child link="estop_button"/>
+    <origin rpy="0 1.5708 0" xyz="0.16 0.0 0.075"/>
+  </joint>
 </robot>

Commit message: added new tf xacro

File: missions/params/giraff.xacro (robot description, xacro)
@@ -32,5 +32,5 @@
   </material>
   # Base
-  <link name="base_link">
+  <link name="$(arg frame_ns)_base_link">
     <visual>
       <geometry>
@@ -41,6 +41,11 @@
     </visual>
   </link>
+  <joint name="$(arg frame_ns)_base_footprint_to_base_link" type="fixed">
+      <parent link="$(arg frame_ns)_base_footprint"/>
+      <child link="$(arg frame_ns)_base_link"/>
+      <origin rpy="0 0 0" xyz="0 0.24 0.10"/>             # Displacement/rotation of the reference_link with respect parent reference_link (TF)
+    </joint>
   # Left wheel
-  <link name="left_wheel">
+  <link name="$(arg frame_ns)_left_wheel">
     <visual>
       <origin rpy="1.57075 0 0" xyz="0 0 0"/>           # Displacement/rotation of the part center with respect the reference_link
@@ -51,11 +56,11 @@
     </visual>
   </link>
-  <joint name="base_to_left_wheel_joint" type="fixed">
-    <parent link="base_link"/>
-    <child link="left_wheel"/>
+  <joint name="$(arg frame_ns)_base_to_left_wheel_joint" type="fixed">
+    <parent link="$(arg frame_ns)_base_link"/>
+    <child link="$(arg frame_ns)_left_wheel"/>
     <origin rpy="0 0 0" xyz="0 0.24 0.10"/>             # Displacement/rotation of the reference_link with respect parent reference_link (TF)
   </joint>
   # Right wheel
-  <link name="right_wheel">
+  <link name="$(arg frame_ns)_right_wheel">
     <visual>
       <origin rpy="1.57075 0 0" xyz="0 0 0"/>           # Displacement/rotation of the part center with respect the reference_link
@@ -66,7 +71,7 @@
     </visual>
   </link>
-  <joint name="base_to_right_wheel_joint" type="fixed">
-    <parent link="base_link"/>
-    <child link="right_wheel"/>
+  <joint name="$(arg frame_ns)_base_to_right_wheel_joint" type="fixed">
+    <parent link="$(arg frame_ns)_base_link"/>
+    <child link="$(arg frame_ns)_right_wheel"/>
     <origin rpy="0 0 0" xyz="0 -0.24 0.10"/>            # Displacement/rotation of the reference_link with respect parent reference_link (TF)
   </joint>

Commit message: added new tf xacro

File: missions/params/giraff.xacro (robot description, xacro)
@@ -32,4 +32,7 @@
   </material>
   # Base
+  <link name="$(arg frame_ns)_base_footprint">
+  </link>
+  # Base
   <link name="$(arg frame_ns)_base_link">
     <visual>

Commit message: fixed xacro

File: missions/params/giraff.xacro (robot description, xacro)
@@ -47,6 +47,6 @@
       <parent link="$(arg frame_ns)_base_footprint"/>
       <child link="$(arg frame_ns)_base_link"/>
-      <origin rpy="0 0 0" xyz="0 0.24 0.10"/>             # Displacement/rotation of the reference_link with respect parent reference_link (TF)
-    </joint>
+      <origin rpy="0 0 0" xyz="0 0 0.10"/>             # Displacement/rotation of the reference_link with respect parent reference_link (TF)
+  </joint>
   # Left wheel
   <link name="$(arg frame_ns)_left_wheel">
@@ -155,5 +155,5 @@
   </joint>
   # Hokuyo front
-  <link name="laser_link">
+  <link name="$(arg frame_ns)_laser_link">
     <visual>
       <geometry>
@@ -165,7 +165,7 @@
   </link>
   <joint name="base_link_to_laser_link" type="fixed">
-    <parent link="base_link"/>
-    <child link="laser_link"/>
-    <origin rpy="0 0 0" xyz="0.2062 0.0 0.0"/>     # Set Manually z=0.28
+    <parent link="$(arg frame_ns)_base_link"/>
+    <child link="$(arg frame_ns)_laser_link"/>
+    <origin rpy="0 0 0" xyz="0.2062 0.0 0.28"/>     # Set Manually z=0.28
   </joint>
   # RGBD_DOWN

Commit message: fixed xacro

File: missions/params/giraff.xacro (robot description, xacro)
@@ -31,6 +31,8 @@
     <color rgba="0.0 0.9 0.0 1"/>
   </material>
-  # Base
+  # Base footprint
   <link name="$(arg frame_ns)_base_footprint">
+    <visual>
+     </visual>
   </link>
   # Base

Commit message: fixed xacro

File: missions/params/giraff.xacro (robot description, xacro)
@@ -34,4 +34,5 @@
   <link name="$(arg frame_ns)_base_footprint">
     <visual>
+    <origin rpy="0 0 0" xyz="0 0 0"/>
      </visual>
   </link>

Commit message: fixed xacro

File: missions/params/giraff.xacro (robot description, xacro)
@@ -167,5 +167,5 @@
     </visual>
   </link>
-  <joint name="base_link_to_laser_link" type="fixed">
+  <joint name="$(arg frame_ns)_base_link_to_laser_link" type="fixed">
     <parent link="$(arg frame_ns)_base_link"/>
     <child link="$(arg frame_ns)_laser_link"/>

Commit message: remove tf from giraff driver node

File: missions/params/giraff.xacro (robot description, xacro)
@@ -82,79 +82,4 @@
     <origin rpy="0 0 0" xyz="0 -0.24 0.10"/>            # Displacement/rotation of the reference_link with respect parent reference_link (TF)
   </joint>
-  # Body
-  <link name="body">
-    <visual>
-      <geometry>
-        <box size="0.30 0.20 0.45"/>
-      </geometry>
-      <material name="body_color"/>
-    </visual>
-  </link>
-  <joint name="base_to_body" type="fixed">
-    <parent link="base_link"/>
-    <child link="body"/>
-    <origin xyz="0.0 0.0 0.455"/>
-  </joint>
-  # Neck (this tf is considered fixed)
-  <link name="neck">
-    <visual>
-      <geometry>
-        <box size="0.05 0.05 0.41"/>
-      </geometry>
-      <material name="grey"/>
-    </visual>
-  </link>
-  <joint name="body_to_neck" type="fixed">
-    <parent link="body"/>
-    <child link="neck"/>
-    <origin xyz="0.0 0.0 0.43"/>
-  </joint>
-  # Head
-  <link name="head">
-    <visual>
-      <geometry>
-        <box size="0.05 0.30 0.56"/>
-      </geometry>
-      <material name="body_color"/>
-    </visual>
-  </link>
-  <joint name="neck_to_head" type="fixed">
-    <parent link="neck"/>
-    <child link="head"/>
-    <origin xyz="0 0 0.485"/>
-  </joint>
-  # Screen (this tf is published by the giraff_ros_driver using Tilt)
-  <link name="screen">
-    <visual>
-      <geometry>
-        <box size="0.05 0.22 0.40"/>
-      </geometry>
-      <material name="white"/>
-    </visual>
-  </link>
-  <joint name="neck_to_screen" type="revolute">
-    <parent link="head"/>
-    <child link="screen"/>
-    <axis xyz="0 1 0"/>
-    <limit effort="1000.0" lower="-2.094395102" upper="2.094395102" velocity="0.5"/>
-    <origin rpy="0 0 0" xyz="0.02 0.0 0.0"/>
-  </joint>
-  ## SENSORS AND ACTUATORS ##
-  #=========================#
-  # FISH_EYE
-  <link name="usb_camera_link">
-    <visual>
-      <geometry>
-        <cylinder length="0.02" radius="0.02"/>
-      </geometry>
-      <material name="black"/>
-      <origin rpy="0 1.57079 0" xyz="0 0.0 0.0"/>     # Displacement/Rotation of the center with respect usb_camera_link
-    </visual>
-  </link>
-  <joint name="screen_to_usb_camera_link" type="fixed">
-    <parent link="screen"/>
-    <child link="usb_camera_link"/>
-    <origin rpy="0 0.3927 0" xyz="0.05 0.0 0.20"/>
-  </joint>
   # Hokuyo front
   <link name="$(arg frame_ns)_laser_link">
@@ -172,78 +97,3 @@
     <origin rpy="0 0 0" xyz="0.2062 0.0 0.28"/>     # Set Manually z=0.28
   </joint>
-  # RGBD_DOWN
-  # For ASTRA rgbd cameras ref_link is located 10cm in y-axis
-  <link name="camera_down_link">
-    <visual>
-      <geometry>
-        <box size="0.04 0.16 0.03"/>
-      </geometry>
-      <material name="black"/>
-      <origin rpy="0 0 0" xyz="0 -0.10 0.0"/>     # Displacement/Rotation of the center with respect camera_down_link
-    </visual>
-  </link>
-  <joint name="base_link_to_camera_down_link" type="fixed">
-    <parent link="base_link"/>
-    <child link="camera_down_link"/>
-    <origin rpy="0 -0.2 0" xyz="0.06 0.10 0.985"/>     # Manually set
-  </joint>
-  # RGBD_UP
-  # For ASTRA rgbd cameras ref_link is located 10cm in y-axis
-  <link name="camera_up_link">
-    <visual>
-      <geometry>
-        <box size="0.04 0.16 0.03"/>
-      </geometry>
-      <material name="black"/>
-      <origin rpy="0 0 0" xyz="0 -0.06 0.0"/>     # Displacement/Rotation of the center with respect camera_up_link
-    </visual>
-  </link>
-  <joint name="base_link_to_camera_up_link" type="fixed">
-    <parent link="base_link"/>
-    <child link="camera_up_link"/>
-    <!-- <origin rpy="0 0.8 0" xyz="0.09 0.10 1.65"/> -->     # Manually set
-    <origin rpy="0.0062 0.7527 0" xyz="0.09 0.06 1.5737"/>             # Calibration
-  </joint>
-  # red button
-  <link name="red_button">
-    <visual>
-      <geometry>
-        <cylinder length="0.02" radius="0.03"/>
-      </geometry>
-      <material name="red"/>
-    </visual>
-  </link>
-  <joint name="body_to_red_button" type="fixed">
-    <parent link="body"/>
-    <child link="red_button"/>
-    <origin xyz="0.11 0.05 0.225"/>
-  </joint>
-  # green button
-  <link name="green_button">
-    <visual>
-      <geometry>
-        <cylinder length="0.02" radius="0.03"/>
-      </geometry>
-      <material name="green"/>
-    </visual>
-  </link>
-  <joint name="body_to_green_button" type="fixed">
-    <parent link="body"/>
-    <child link="green_button"/>
-    <origin xyz="0.11 -0.05 0.225"/>
-  </joint>
-  # e-stop button
-  <link name="estop_button">
-    <visual>
-      <geometry>
-        <cylinder length="0.02" radius="0.02"/>
-      </geometry>
-      <material name="red"/>
-    </visual>
-  </link>
-  <joint name="body_to_estop_button" type="fixed">
-    <parent link="body"/>
-    <child link="estop_button"/>
-    <origin rpy="0 1.5708 0" xyz="0.16 0.0 0.075"/>
-  </joint>
 </robot>

Commit message: remove tf from giraff driver node

File: missions/params/giraff.xacro (robot description, xacro)
@@ -44,5 +44,5 @@
       </geometry>
       <material name="body_color"/>
-      <origin rpy="0 0 0" xyz="0 0 0.13"/>              # Displacement/rotation of the part center with respect the reference_link (base_link)
+      <origin rpy="0 0 0" xyz="0 0 0"/>              # Displacement/rotation of the part center with respect the reference_link (base_link)
     </visual>
   </link>

Commit message: remove tf from giraff driver node

File: missions/params/giraff.xacro (robot description, xacro)
@@ -44,5 +44,5 @@
       </geometry>
       <material name="body_color"/>
-      <origin rpy="0 0 0" xyz="0 0 0"/>              # Displacement/rotation of the part center with respect the reference_link (base_link)
+      <origin rpy="0 0 0" xyz="0 0 0.02"/>              # Displacement/rotation of the part center with respect the reference_link (base_link)
     </visual>
   </link>
@@ -50,5 +50,5 @@
       <parent link="$(arg frame_ns)_base_footprint"/>
       <child link="$(arg frame_ns)_base_link"/>
-      <origin rpy="0 0 0" xyz="0 0 0.10"/>             # Displacement/rotation of the reference_link with respect parent reference_link (TF)
+      <origin rpy="0 0 0" xyz="0 0 0"/>             # Displacement/rotation of the reference_link with respect parent reference_link (TF)
   </joint>
   # Left wheel
