Commit message: fixed xacro giraff

File: missions/params/giraff.xacro (robot description, xacro)
@@ -44,5 +44,5 @@
       </geometry>
       <material name="body_color"/>
-      <origin rpy="0 0 0" xyz="0 0 0.02"/>              # Displacement/rotation of the part center with respect the reference_link (base_link)
+      <origin rpy="0 0 0" xyz="0 0 0.10"/>              # Displacement/rotation of the part center with respect the reference_link (base_link)
     </visual>
   </link>
@@ -50,5 +50,5 @@
       <parent link="$(arg frame_ns)_base_footprint"/>
       <child link="$(arg frame_ns)_base_link"/>
-      <origin rpy="0 0 0" xyz="0 0 0"/>             # Displacement/rotation of the reference_link with respect parent reference_link (TF)
+      <origin rpy="0 0 0" xyz="0 0 0.03"/>             # Displacement/rotation of the reference_link with respect parent reference_link (TF)
   </joint>
   # Left wheel
@@ -65,5 +65,5 @@
     <parent link="$(arg frame_ns)_base_link"/>
     <child link="$(arg frame_ns)_left_wheel"/>
-    <origin rpy="0 0 0" xyz="0 0.24 0.10"/>             # Displacement/rotation of the reference_link with respect parent reference_link (TF)
+    <origin rpy="0 0 0" xyz="0 0.24 0.07"/>             # Displacement/rotation of the reference_link with respect parent reference_link (TF)
   </joint>
   # Right wheel
@@ -80,5 +80,5 @@
     <parent link="$(arg frame_ns)_base_link"/>
     <child link="$(arg frame_ns)_right_wheel"/>
-    <origin rpy="0 0 0" xyz="0 -0.24 0.10"/>            # Displacement/rotation of the reference_link with respect parent reference_link (TF)
+    <origin rpy="0 0 0" xyz="0 -0.24 0.07"/>            # Displacement/rotation of the reference_link with respect parent reference_link (TF)
   </joint>
   # Hokuyo front
@@ -95,5 +95,95 @@
     <parent link="$(arg frame_ns)_base_link"/>
     <child link="$(arg frame_ns)_laser_link"/>
-    <origin rpy="0 0 0" xyz="0.2062 0.0 0.28"/>     # Set Manually z=0.28
+    <origin rpy="0 0 0" xyz="0.2062 0.0 0.25"/>     # Set Manually z=0.28
   </joint>
+  # Body
+  <link name="$(arg frame_ns)_body">
+    <visual>
+      <geometry>
+        <box size="0.30 0.20 0.45"/>
+      </geometry>
+      <material name="body_color"/>
+    </visual>
+  </link>
+  <joint name="$(arg frame_ns)_base_to_body" type="fixed">
+    <parent link="$(arg frame_ns)_base_link"/>
+    <child link="$(arg frame_ns)_body"/>
+    <origin xyz="0.0 0.0 0.42"/>
+  </joint>
+  # Neck (this tf is considered fixed)
+  <link name="$(arg frame_ns)_neck">
+    <visual>
+      <geometry>
+        <box size="0.05 0.05 0.30"/>
+      </geometry>
+      <material name="grey"/>
+    </visual>
+  </link>
+  <joint name="$(arg frame_ns)_body_to_neck" type="fixed">
+    <parent link="$(arg frame_ns)_body"/>
+    <child link="$(arg frame_ns)_neck"/>
+    <origin xyz="0.0 0.0 0.375"/>
+  </joint>
+  # Head
+  <link name="$(arg frame_ns)_head">
+    <visual>
+      <geometry>
+        <box size="0.05 0.30 0.56"/>
+      </geometry>
+      <material name="body_color"/>
+    </visual>
+  </link>
+  <joint name="$(arg frame_ns)_neck_to_head" type="fixed">
+    <parent link="$(arg frame_ns)_neck"/>
+    <child link="$(arg frame_ns)_head"/>
+    <origin xyz="0 0 0.43"/>
+  </joint>
+  # Screen (this tf is published by the giraff_ros_driver using Tilt)
+  <link name="$(arg frame_ns)_screen">
+    <visual>
+      <geometry>
+        <box size="0.05 0.22 0.40"/>
+      </geometry>
+      <material name="white"/>
+    </visual>
+  </link>
+  <joint name="$(arg frame_ns)_neck_to_screen" type="revolute">
+    <parent link="$(arg frame_ns)_head"/>
+    <child link="$(arg frame_ns)_screen"/>
+    <axis xyz="0 1 0"/>
+    <limit effort="1000.0" lower="-2.094395102" upper="2.094395102" velocity="0.5"/>
+    <origin rpy="0 0 0" xyz="0.02 0.0 0.0"/>
+  </joint>
+  # Camera down
+  <link name="$(arg frame_ns)_camera_down_link">
+      <visual>
+        <geometry>
+          <box size="0.04 0.16 0.03"/>
+        </geometry>
+        <material name="black"/>
+        <origin rpy="0 0 0" xyz="0 0 0.0"/>     # Displacement/Rotation of the center with respect camera_down_link
+      </visual>
+    </link>
+    <joint name="$(arg frame_ns)_base_link_to_camera_down_link" type="fixed">
+      <parent link="$(arg frame_ns)_base_link"/>
+      <child link="$(arg frame_ns)_camera_down_link"/>
+      <origin rpy="0 -0.2 0" xyz="0.06 0.0 0.88"/>     # Manually set
+    </joint>
+ # RGBD_UP
+    # For ASTRA rgbd cameras ref_link is located 10cm in y-axis
+    <link name="$(arg frame_ns)_camera_up_link">
+      <visual>
+        <geometry>
+          <box size="0.04 0.16 0.03"/>
+        </geometry>
+        <material name="black"/>
+        <origin rpy="0 0 0" xyz="0 0 0.0"/>     # Displacement/Rotation of the center with respect camera_up_link
+      </visual>
+    </link>
+    <joint name="$(arg frame_ns)_base_link_to_camera_up_link" type="fixed">
+      <parent link="$(arg frame_ns)_base_link"/>
+      <child link="$(arg frame_ns)_camera_up_link"/>
+      <!-- <origin rpy="0 0.8 0" xyz="0.09 0.10 1.65"/> -->     # Manually set
+      <origin rpy="0.0062 0.7527 0" xyz="0.06 0.0 1.4737"/>             # Calibration
+    </joint>
 </robot>

Commit message: fixed tf

File: missions/params/giraff.xacro (robot description, xacro)
@@ -165,9 +165,4 @@
       </visual>
     </link>
-    <joint name="$(arg frame_ns)_base_link_to_camera_down_link" type="fixed">
-      <parent link="$(arg frame_ns)_base_link"/>
-      <child link="$(arg frame_ns)_camera_down_link"/>
-      <origin rpy="0 -0.2 0" xyz="0.06 0.0 0.88"/>     # Manually set
-    </joint>
  # RGBD_UP
     # For ASTRA rgbd cameras ref_link is located 10cm in y-axis
@@ -181,9 +176,3 @@
       </visual>
     </link>
-    <joint name="$(arg frame_ns)_base_link_to_camera_up_link" type="fixed">
-      <parent link="$(arg frame_ns)_base_link"/>
-      <child link="$(arg frame_ns)_camera_up_link"/>
-      <!-- <origin rpy="0 0.8 0" xyz="0.09 0.10 1.65"/> -->     # Manually set
-      <origin rpy="0.0062 0.7527 0" xyz="0.06 0.0 1.4737"/>             # Calibration
-    </joint>
 </robot>

Commit message: fixed tf

File: missions/params/giraff.xacro (robot description, xacro)
@@ -151,6 +151,4 @@
     <parent link="$(arg frame_ns)_head"/>
     <child link="$(arg frame_ns)_screen"/>
-    <axis xyz="0 1 0"/>
-    <limit effort="1000.0" lower="-2.094395102" upper="2.094395102" velocity="0.5"/>
     <origin rpy="0 0 0" xyz="0.02 0.0 0.0"/>
   </joint>

Commit message: fixed tf

File: missions/params/giraff.xacro (robot description, xacro)
@@ -148,5 +148,5 @@
     </visual>
   </link>
-  <joint name="$(arg frame_ns)_neck_to_screen" type="revolute">
+  <joint name="$(arg frame_ns)_head_to_screen" type="fixed">
     <parent link="$(arg frame_ns)_head"/>
     <child link="$(arg frame_ns)_screen"/>

Commit message: fixed tf

File: missions/params/giraff.xacro (robot description, xacro)
@@ -163,4 +163,9 @@
       </visual>
     </link>
+    <joint name="$(arg frame_ns)_base_link_to_camera_down_link" type="fixed">
+          <parent link="$(arg frame_ns)_base_link"/>
+          <child link="$(arg frame_ns)_camera_down_link"/>
+          <origin rpy="0 -0.2 0" xyz="0.06 0.0 0.88"/>     # Manually set
+        </joint>
  # RGBD_UP
     # For ASTRA rgbd cameras ref_link is located 10cm in y-axis
@@ -174,3 +179,9 @@
       </visual>
     </link>
+   <joint name="$(arg frame_ns)_base_link_to_camera_up_link" type="fixed">
+         <parent link="$(arg frame_ns)_base_link"/>
+         <child link="$(arg frame_ns)_camera_up_link"/>
+         <!-- <origin rpy="0 0.8 0" xyz="0.09 0.10 1.65"/> -->     # Manually set
+         <origin rpy="0.0062 0.7527 0" xyz="0.06 0.0 1.4737"/>             # Calibration
+       </joint>
 </robot>
